File: controller-pcb/kinBP.kicad_pcb (KiCad board)
At the start: 2 copper layers, 100 x 86.5 mm, 30 parts, among them J1 LEFT_TOP, J10 LEFT_THUMB, J11 RIGHT_THUMB, J12 RIGHT_THUMB, J13 LEFT_THUMB, J2 LEFT_TOP, J3 RIGHT_TOP, J4 RIGHT_TOP, J5 RIGHT_KEYWELL, J6 LEFT_KEYWELL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

Commit message: Original commit
Parts:
- removed G1: LOGO, logo:q64logo
- removed J12: RIGHT_THUMB, Connector_Molex:Molex_PicoBlade_53048-0710_1x07_P1.25mm_Horizontal
- removed J13: LEFT_THUMB, Connector_Molex:Molex_PicoBlade_53048-0710_1x07_P1.25mm_Horizontal
- removed J7: LEFT_THUMB, Connector_PinHeader_2.54mm:PinHeader_1x10_P2.54mm_Vertical
- removed J8: RIGHT_THUMB, Connector_PinHeader_2.54mm:PinHeader_1x10_P2.54mm_Vertical
- moved G*** 20.2 mm to (141.2, 65.7)
Routing:
- net COL_5: track 242.5 -> 211.9 mm
- net ROW_2: track 142.2 -> 122.0 mm
- net ROW_4: track 69.0 -> 49.6 mm
- net ROW_5: track 75.8 -> 61.1 mm
- net ROW_9: track 76.3 -> 61.8 mm
- net COL_6: track 165.4 -> 152.7 mm, vias 0 -> 1
- net ROW_6: track 104.6 -> 94.1 mm, vias 0 -> 2
- net ROW_3: track 97.1 -> 92.0 mm
- net ROW_0: track 111.9 -> 116.2 mm
- net ROW_7: track 71.9 -> 67.7 mm
- net LED_KPD: track 63.5 -> 65.5 mm
Other:
- board text added: "Based on KinBP v1.21"
- board text added: "KinTwin v1.0"
- board text removed: "KinBP v1.21"
- board text removed: "Open Hardware: CC-BY-SA"
- board text removed: "github.com/DmNosachev/kinbp"
